Commit message: Working on Kinova arm fo bci

File: rlsimenv/data/cube2.urdf (robot description, URDF)
Before this commit: robot cube.urdf, 1 links, 0 joints
Links:
- link baseLink: mass .1 -> 1.1

File: rlsimenv/data/disk.urdf (robot description, URDF)
Before this commit: robot cube.urdf, 1 links, 0 joints
Links:
- link baseLink: geometry collision cylinder length=0.5 radius=2.0; visual cylinder length=0.5 radius=2.0
