Commit message: Roof; N particles; No collision; z-velocity zeroing; vel. clamping

File: rlsimenv/data/door_cube.urdf (robot description, URDF)
Before this commit: robot door_cube.urdf, 1 links, 0 joints
Links:
- link baseLink: geometry collision box size=0.2 1.0 1.0; visual mesh filename=cube.obj scale=0.2 1.0 1.0
