Commit message: Working on objects sim

File: rlsimenv/data/sphere2_red2.urdf (robot description, URDF)
Before this commit: robot door_cube.urdf, 1 links, 0 joints
Links:
- link baseLink: mass 5.1 -> 1.0; geometry collision sphere radius=0.5; visual mesh filename=sphere_smooth.obj scale=0.5 0.5 0.5
